File: KC1FSZ-Converter-1.kicad_pcb (KiCad board)
At the start: 2 copper layers, 50 x 30 mm, 26 parts, among them J1 Conn_02x05_Odd_Even, J2 Conn_01x02, J3 Conn_02x02_Odd_Even, U1 BGA2867, U2 PAT1220-C-6DB, U3 MASW-007221, U4 ADE-1+, U5 MASW-007221, U6 BGA2867, U7 PAT1220-C-6DB

Commit message: Ready for RIT
Parts:
- J3: value Conn_02x02_Odd_Even -> Conn_02x03_Odd_Even; footprint Connector_PinHeader_2.54mm:PinHeader_2x02_P2.54mm_Vertical -> Connector_PinHeader_2.54mm:PinHeader_2x03_P2.54mm_Vertical
- moved J3 2.00 mm to (157.0, 75.0)
- moved RV1 1.00 mm to (151.5, 75.0)
- moved C11 0.71 mm to (144.5, 76.0)
- moved J2 0.50 mm to (143.0, 72.5)
Connections:
- C9 pad 1: +5VA -> +5VD
- U6 pad 1: +5VA -> +5VD
Routing:
- net +5VA: track 63.4 -> 11.5 mm
- net +5VD: track 0.00 -> 36.9 mm
- net SEL1: track 34.5 -> 36.9 mm
- net RX_IN: track 3.68 -> 5.12 mm
- net GNDA: track 15.5 -> 16.8 mm, vias 9 -> 24
- net LO_IN: track 3.20 -> 3.70 mm
